File: PCB fuse box.kicad_pcb (KiCad board)
At the start: 2 copper layers, 115.6 x 62 mm, 21 parts, among them J1 6570XX230201_657012230201, J2 6570XX230201_657012230201, J3 449140201, K1 AZ2150-1A-12DEF, K2 AZ2150-1A-12DEF

Commit message: Fixed
Connections:
- H4 pad 1: (no net) -> GND
Routing:
- net relay2: track 50.1 -> 51.5 mm
- net 8: track 39.7 -> 38.6 mm
Changed lines of the file:
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@@
 			(layers "*.Cu" "*.Mask")
 			(remove_unused_layers no)
+			(net "GND")
 			(zone_connect 2)
 		)
@@
 	)
 	(segment
-		(start 95.4044 86.0044)
-		(end 117.172801 86.0044)
-		(width 0.3)
+		(start 90.145 109.855)
+		(end 84.582 109.855)
+		(width 0.6)
 		(layer "F.Cu")
 		(net "relay2")
 	)
 	(segment
-		(start 84.582 109.855)
-		(end 95.4 99.037)
-		(width 0.3)
+		(start 92 92.5)
+		(end 92 108)
+		(width 0.6)
 		(layer "F.Cu")
 		(net "relay2")
 	)
 	(segment
-		(start 95.4 86)
-		(end 95.4044 86.0044)
-		(width 0.3)
+		(start 117.172801 86.0044)
+		(end 98.4956 86.0044)
+		(width 0.6)
 		(layer "F.Cu")
 		(net "relay2")
 	)
 	(segment
-		(start 95.4 99.037)
-		(end 95.4 86)
-		(width 0.3)
+		(start 92 108)
+		(end 90.145 109.855)
+		(width 0.6)
+		(layer "F.Cu")
+		(net "relay2")
+	)
+	(segment
+		(start 98.4956 86.0044)
+		(end 92 92.5)
+		(width 0.6)
 		(layer "F.Cu")
 		(net "relay2")
@@
 	)
 	(segment
-		(start 128.2 77.216)
-		(end 128.2 76.1)
-		(width 2)
-		(layer "B.Cu")
-		(net "8")
-	)
-	(segment
-		(start 128.25 75.6)
+		(start 156.516 73.2)
 		(end 130.65 73.2)
-		(width 2)
-		(layer "B.Cu")
-		(net "8")
-	)
-	(segment
-		(start 130.65 73.2)
-		(end 156.516 73.2)
 		(width 2)
 		(layer "B.Cu")
@@
 		(width 2)
 		(layer "B.Cu")
+		(net "8")
+	)
+	(segment
+		(start 130.65 73.2)
+		(end 128.25 75.6)
+		(width 2)
+		(layer "B.Cu")

Commit message: fix smth
Parts:
- removed H4: MountingHole, MountingHole:MountingHole_2.2mm_M2_Pad
- added J4: 449140201, fuse relay box:CONN_SD-44914-002_02_MOL, F.Cu at (131.0, 86.0)
Routing:
- net 10: track 79.8 -> 80.9 mm
- net relay1: track 39.0 -> 38.3 mm
Changed lines of the file:
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@@
 			(outputformat 1)
 			(mirror no)
-			(drillshape 1)
+			(drillshape 0)
 			(scaleselection 1)
-			(outputdirectory "")
+			(outputdirectory "../order/Production/Fuse/")
 		)
 	)
@@
 		(embedded_fonts no)
 	)
-	(footprint "MountingHole:MountingHole_2.2mm_M2_Pad"
-		(layer "F.Cu")
-		(at 84.8 98.7)
-		(descr "Mounting Hole 2.2mm, M2, generated by kicad-footprint-generator mountinghole.py")
-		(tags "mountinghole M2")
-		(property "Reference" "H4"
-			(at 0 -3.15 0)
-			(layer "F.SilkS")
-			(effects
-				(font
-					(size 1 1)
-					(thickness 0.15)
-				)
-			)
-		)
-		(property "Value" "MountingHole"
-			(at 0 3.15 0)
-			(layer "F.Fab")
-			(effects
-				(font
-					(size 1 1)
-					(thickness 0.15)
-				)
-			)
-		)
-		(property "Datasheet" ""
-			(at 0 0 0)
-			(layer "F.Fab")
-			(hide yes)
-			(effects
-				(font
-					(size 1.27 1.27)
-				)
-			)
-		)
-		(property "Description" "Mounting Hole without connection"
-			(at 0 0 0)
-			(layer "F.Fab")
-			(hide yes)
-			(effects
-				(font
-					(size 1.27 1.27)
-				)
-			)
-		)
-		(property ki_fp_filters "MountingHole*")
-		(sheetname "/")
-		(sheetfile "PCB fuse box.kicad_sch")
-		(units
-			(unit
-				(name "A")
-				(pins)
-			)
-		)
-		(attr exclude_from_bom)
-		(duplicate_pad_numbers_are_jumpers no)
-		(fp_circle
-			(center 0 0)
-			(end 2.2 0)
-			(stroke
-				(width 0.15)
-				(type solid)
-			)
-			(fill no)
-			(layer "Cmts.User")
-		)
-		(fp_circle
-			(center 0 0)
-			(end 2.45 0)
-			(stroke
-				(width 0.05)
-				(type solid)
-			)
-			(fill no)
-			(layer "F.CrtYd")
-		)
-		(fp_text user "${REFERENCE}"
-			(at 0 0 0)
-			(layer "F.Fab")
-			(effects
-				(font
-					(size 1 1)
-					(thickness 0.15)
-				)
-			)
-		)
-		(pad "1" thru_hole circle
-			(at 0 0)
-			(size 4.4 4.4)
-			(drill 2.2)
-			(layers "*.Cu" "*.Mask")
-			(remove_unused_layers no)
-			(net "GND")
-			(zone_connect 2)
-		)
-		(embedded_fonts no)
-	)
 	(footprint "Fuse:Fuse_Blade_ATO_directSolder"
 		(layer "F.Cu")
@@
 		)
 	)
+	(footprint "fuse relay box:CONN_SD-44914-002_02_MOL"
+		(layer "F.Cu")
+		(at 131 86.0334 90)
+		(tags "449140201 ")
+		(property "Reference" "J4"
+			(at 0 -1.5 90)
+			(unlocked yes)
+			(layer "F.SilkS")
+			(effects
+				(font
+					(size 1 1)
+					(thickness 0.15)
+				)
+			)
+		)
+		(property "Value" "449140201"
+			(at 0 0 90)
+			(unlocked yes)
+			(layer "F.Fab")
+			(effects
+				(font
+					(size 1 1)
+					(thickness 0.15)
+				)
+			)
+		)
+		(property "Datasheet" "https://www.molex.com/en-us/products/part-detail-pdf/449140201?display=pdf"
+			(at 0 0 90)
+			(layer "F.Fab")
+			(hide yes)
+			(effects
+				(font
+					(size 1.27 1.27)
+				)
+			)
+		)
+		(property "Description" ""
+			(at 0 0 90)
+			(layer "F.Fab")
+			(hide yes)
+			(effects
+				(font
+					(size 1.27 1.27)
+				)
+			)
+		)
+		(property ki_fp_filters "CONN_SD-44914-002_02_MOL")
+		(sheetname "/")
+		(sheetfile "PCB fuse box.kicad_sch")
+		(attr through_hole)
+		(duplicate_pad_numbers_are_jumpers no)
+		(fp_line
+			(start 3.7084 -6.457)
+			(end -3.7084 -6.457)
+			(stroke
+				(width 0.1524)
+				(type solid)
+			)
+			(layer "F.SilkS")
+		)
+		(fp_line
+			(start -3.7084 -6.457)
+			(end -3.7084 -4.460126)
+			(stroke
+				(width 0.1524)
+				(type solid)
+			)
+			(layer "F.SilkS")
+		)
+		(fp_line
+			(start 3.7084 -4.460126)
+			(end 3.7084 -6.457)
+			(stroke
+				(width 0.1524)
+				(type solid)
+			)
+			(layer "F.SilkS")
+		)
+		(fp_line
+			(start -3.7084 -3.419873)
+			(end -3.7084 2.5854)
+			(stroke
+				(width 0.1524)
+				(type solid)
+			)
+			(layer "F.SilkS")
+		)
+		(fp_line
+			(start 3.7084 2.5854)
+			(end 3.7084 -3.419873)
+			(stroke
+				(width 0.1524)
+				(type solid)
+			)
+			(layer "F.SilkS")
+		)
+		(fp_line
+			(start -3.7084 2.5854)
+			(end 3.7084 2.5854)
+			(stroke
+				(width 0.1524)
+				(type solid)
+			)
+			(layer "F.SilkS")
+		)
+		(fp_circle
+			(center 4.3434 0)
+			(end 4.7244 0)
+			(stroke
+				(width 0.508)
+				(type solid)
+			)
+			(fill no)
+			(layer "F.SilkS")
+		)
+		(fp_circle
+			(center 4.3434 0)
+			(end 4.7244 0)
+			(stroke
+				(width 0.508)
+				(type solid)
+			)
+			(fill no)
+			(layer "B.SilkS")
+		)
+		(fp_line
+			(start 3.8354 -6.584)
+			(end -3.8354 -6.584)
+			(stroke
+				(width 0.1524)
+				(type solid)
+			)
+			(layer "F.CrtYd")
+		)
+		(fp_line
+			(start -3.8354 -6.584)
+			(end -3.8354 2.7124)
+			(stroke
+				(width 0.1524)
+				(type solid)
+			)
+			(layer "F.CrtYd")
+		)
+		(fp_line
+			(start 3.8354 2.7124)
+			(end 3.8354 -6.584)
+			(stroke
+				(width 0.1524)
+				(type solid)
+			)
+			(layer "F.CrtYd")
+		)
+		(fp_line
+			(start -3.8354 2.7124)
+			(end 3.8354 2.7124)
+			(stroke
+				(width 0.1524)
+				(type solid)
+			)
+			(layer "F.CrtYd")
+		)
+		(fp_line
+			(start 3.5814 -6.33)
+			(end -3.5814 -6.33)
+			(stroke
+				(width 0.0254)
+				(type solid)
+			)
+			(layer "F.Fab")
+		)
+		(fp_line
+			(start -3.5814 -6.33)
+			(end -3.5814 2.4584)
+			(stroke
+				(width 0.0254)
+				(type solid)
+			)
+			(layer "F.Fab")
+		)
+		(fp_line
+			(start 3.5814 2.4584)
+			(end 3.5814 -6.33)
+			(stroke
+				(width 0.0254)
+				(type solid)
+			)
+			(layer "F.Fab")
+		)
+		(fp_line
+			(start -3.5814 2.4584)
+			(end 3.5814 2.4584)
+			(stroke
+				(width 0.0254)
+				(type solid)
+			)
+			(layer "F.Fab")
+		)
+		(fp_circle
+			(center 0 1.905)
+			(end 0.381 1.905)
+			(stroke
+				(width 0.508)
+				(type solid)
+			)
+			(fill no)
+			(layer "F.Fab")
+		)
+		(fp_text user "${REFERENCE}"
+			(at 0 -1.5 90)
+			(unlocked yes)
+			(layer "F.Fab")
+			(effects
+				(font
+					(size 1 1)
+					(thickness 0.15)
+				)
+			)
+		)
+		(pad "" np_thru_hole circle
+			(at -3.000002 -3.94 90)
+			(size 1.0922 1.0922)
+			(drill 1.0922)
+			(layers)
+		)
+		(pad "" np_thru_hole circle
+			(at 3.000002 -3.94 90)
+			(size 1.0922 1.0922)
+			(drill 1.0922)
+			(layers)
+		)
+		(pad "1" thru_hole circle
+			(at 0 0 90)
+			(size 1.5748 1.5748)
+			(drill 1.0668)
+			(layers "*.Cu" "*.Mask")
+			(remove_unused_layers no)
+			(pinfunction "1_1")
+			(pintype "unspecified")
+		)
+		(pad "2" thru_hole circle
+			(at 0 -2.999999 90)
+			(size 1.5748 1.5748)
+			(drill 1.0668)
+			(layers "*.Cu" "*.Mask")
+			(remove_unused_layers no)
+			(net "GND")
+			(pinfunction "2_2")
+			(pintype "unspecified")
+		)
+		(embedded_fonts no)
+	)
 	(footprint "Fuse:Fuse_Blade_ATO_directSolder"
 		(layer "F.Cu")
@@
 	)
 	(segment
-		(start 120.1728 86.0044)
-		(end 120.1728 84.890849)
-		(width 0.6)
-		(layer "F.Cu")
-		(net "relay1")
-	)
-	(segment
-		(start 86.534 81.2)
-		(end 84.6328 79.2988)
+		(start 118.6854 84.517)
+		(end 89.851 84.517)
 		(width 0.6)
 		(layer "F.Cu")
@@
 	)
 	(segment
-		(start 120.1728 84.890849)
-		(end 116.481951 81.2)
+		(start 120.1728 86.0044)
+		(end 118.6854 84.517)
 		(width 0.6)
 		(layer "F.Cu")
@@
 	)
 	(segment
-		(start 116.481951 81.2)
-		(end 86.534 81.2)
+		(start 89.851 84.517)
+		(end 84.6328 79.2988)
 		(width 0.6)
 		(layer "F.Cu")
@@
 	)
 	(segment
-		(start 148 76)
-		(end 137.8 76)
+		(start 147.907702 75.991702)
+		(end 148 76.084)
 		(width 2)
 		(layer "B.Cu")
@@
 		(width 2)
 		(layer "B.Cu")
+		(net "10")
+	)
+	(segment
+		(start 136.708298 75.991702)
+		(end 147.907702 75.991702)
+		(width 2)
+		(layer "B.Cu")

Commit message: Add files via upload
Parts:
- F1, F10, F11, F12, F2, F3, F4, F5, F6, F7, F8, F9: footprint Fuse:Fuse_Blade_ATO_directSolder -> fuse-relay_NewFootprints:FUSE_3557-2
- J1, J2: footprint fuse relay box:657012230201 -> fuse-relay_NewFootprints:657012230201
- J3, J4: footprint fuse relay box:CONN_SD-44914-002_02_MOL -> fuse-relay_NewFootprints:CONN_SD-44914-002_02_MOL
- K1, K2: footprint fuse relay box:RELAY_AZ2150-1A-12DEF -> fuse-relay_NewFootprints:RELAY_AZ2150-1A-12DEF
- moved F5 5.41 mm to (123.0, 117.5)
- moved F12 5.36 mm to (123.0, 126.5)
- moved F3 4.34 mm to (143.7, 102.2)
- moved F4 4.34 mm to (152.7, 102.1)
- moved F8 4.34 mm to (134.7, 102.2)
- moved F7 4.34 mm to (125.6, 102.2)
- moved F2 4.34 mm to (170.5, 102.0)
- moved F10 4.34 mm to (188.3, 102.0)
- moved F9 4.34 mm to (179.5, 102.0)
- moved F6 4.34 mm to (116.6, 102.2)
- moved F1 4.34 mm to (161.7, 102.0)
- moved F11 4.07 mm to (123.0, 76.0)
- moved J3 0.17 mm to (120.0, 86.0)
- moved J4 0.17 mm to (130.8, 86.0)
Connections:
- J4 pad 1: (no net) -> GND
- J4 pad 2: GND -> unconnected-(J4-Pad2)
- K1 pad COM: Net-(F11-Pad1) -> Net-(F11-Pad1_1)
Routing:
- net Net-(F11-Pad1_1): track 0.00 -> 22.8 mm
- net Net-(F11-Pad1): track 21.7 -> 0.00 mm
- net 12A: track 35.1 -> 31.3 mm
- net 11: track 29.2 -> 31.0 mm
- net 4: track 12.5 -> 14.1 mm
- net 3A: track 11.8 -> 13.3 mm
- net Net-(F12-Pad1): track 19.1 -> 20.5 mm
- net 11A: track 98.2 -> 99.6 mm
- net 8: track 38.6 -> 40.0 mm
- net 10: track 80.9 -> 82.3 mm
- net 5A: track 13.9 -> 15.1 mm
- net 4A: track 12.6 -> 13.8 mm
- net 7A: track 31.8 -> 32.8 mm
- net 1: track 22.3 -> 21.4 mm
- net 2A: track 12.6 -> 13.3 mm
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
Commit message: fix smth
Parts:
- removed J4: 449140201, fuse-relay_NewFootprints:CONN_SD-44914-002_02_MOL
- added G***: LOGO, logo:logo2, F.Cu at (175.5, 85.0)
- J3: value 449140201 -> 436500315; footprint fuse-relay_NewFootprints:CONN_SD-44914-002_02_MOL -> MOLEX 436500315:CONN_SD-43650-006_03_MOL
- moved J3 1.10 mm to (119.0, 86.5), turned to 180 degrees
Connections:
- J3 pad 1: relay1 -> relay2
- J3 pad 2: relay2 -> relay1
Routing:
- net relay2: track 51.5 -> 44.1 mm
- net relay1: track 38.1 -> 40.3 mm
Other:
- board text added: "Chayanit Soongloy"

Commit message: Adjust width
Routing:
- net 5A: track 15.1 -> 38.1 mm
- net 3: track 14.3 -> 27.2 mm
- net 1A: track 14.6 -> 26.1 mm
- net 6: track 14.9 -> 26.3 mm
- net 5: track 13.6 -> 22.6 mm
- net 2: track 15.5 -> 24.4 mm
- net 9: track 71.0 -> 79.3 mm
- net 4: track 14.1 -> 17.0 mm
- net 2A: track 13.3 -> 16.0 mm
- net 7A: track 32.8 -> 34.2 mm
- net 3A: track 13.3 -> 14.4 mm
- net 4A: track 13.8 -> 14.4 mm
